Commit message: Add .gitignore, update CMakeLists.txt for additional directories, enhance README with setup instructions, modify ur_controllers.yaml for end effector link, create launch file for robot control, and add RViz configuration.

File: urdf/ur_wrapper.xacro (robot description, xacro)
@@ -1,11 +1,13 @@
 <?xml version="1.0"?>
 <robot xmlns:xacro="http://ros.org/wiki/xacro" name="ur_robot">
-    <xacro:property name="ur_type" value="$(arg ur_type)" />
     <!-- Include the standard UR robot -->
     <xacro:include filename="$(find ur_description)/urdf/ur.urdf.xacro" />
-    <xacro:ur_robot ur_type="${ur_type}" prefix="${prefix}" />
-    <!-- Include the blackberry macro-->
-    <xacro:include filename="$(find easy_ur)/urdf/.xacro" />
-    <!-- Call the macro to add probe -->
-    <xacro:add_blackberry />
+    <!-- Include your custom gripper and add the joint to connect to it, then go to the
+    ur_controllers.yaml and change the ee link in the controller parameters -->
+    <!-- <xacro:include filename="$(find gripper_description)/urdf/ur_gripper.xacro" /> -->
+    <!-- <joint name="example_gripper_joint" type="fixed">
+        <parent link="tool0" />
+        <child link="gripper_link" />
+        <origin xyz="0 0 0" rpy="0 0 0" />
+    </joint> -->
 </robot>

Commit message: tested on jazzy

File: urdf/ur_wrapper.xacro (robot description, xacro)
@@ -1,13 +1,60 @@
 <?xml version="1.0"?>
-<robot xmlns:xacro="http://ros.org/wiki/xacro" name="ur_robot">
-    <!-- Include the standard UR robot -->
-    <xacro:include filename="$(find ur_description)/urdf/ur.urdf.xacro" />
-    <!-- Include your custom gripper and add the joint to connect to it, then go to the
+<robot name="ur_robot" xmlns:xacro="http://www.ros.org/wiki/xacro">
+    <!-- Parameters -->
+    <xacro:arg name="ur_type" default="ur20" />
+    <xacro:arg name="joint_limit_parameters_file"
+        default="$(find ur_description)/config/$(arg ur_type)/joint_limits.yaml" />
+    <xacro:arg name="kinematics_parameters_file"
+        default="$(find ur_description)/config/$(arg ur_type)/default_kinematics.yaml" />
+    <xacro:arg name="physical_parameters_file"
+        default="$(find ur_description)/config/$(arg ur_type)/physical_parameters.yaml" />
+    <xacro:arg name="visual_parameters_file"
+        default="$(find ur_description)/config/$(arg ur_type)/visual_parameters.yaml" />
+    <xacro:arg name="robot_ip" default="0.0.0.0" />
+    <xacro:arg name="headless_mode" default="false" />
+    <xacro:arg name="ur_script_filename"
+        default="$(find ur_client_library)/resources/external_control.urscript" />
+    <xacro:arg name="ur_output_recipe_filename"
+        default="$(find ur_robot_driver)/resources/rtde_output_recipe.txt" />
+    <xacro:arg name="ur_input_recipe_filename"
+        default="$(find ur_robot_driver)/resources/rtde_input_recipe.txt" />
+    <xacro:arg name="use_mock_hardware" default="false" />
+    <xacro:arg name="mock_sensor_commands" default="false" />
+    <!-- Include the UR robot macro and ros2_control tag from the driver -->
+    <xacro:include filename="$(find ur_description)/urdf/ur_macro.xacro" />
+    <xacro:include filename="$(find ur_robot_driver)/urdf/ur.ros2_control.xacro" />
+    <!-- URDF root -->
+    <link name="world" />
+    <!-- Instantiate the UR robot -->
+    <xacro:ur_robot
+        name="$(arg ur_type)"
+        tf_prefix="$(arg ur_type)_"
+        parent="world"
+        joint_limits_parameters_file="$(arg joint_limit_parameters_file)"
+        kinematics_parameters_file="$(arg kinematics_parameters_file)"
+        physical_parameters_file="$(arg physical_parameters_file)"
+        visual_parameters_file="$(arg visual_parameters_file)"
+    >
+        <origin xyz="0 0 0" rpy="0 0 0" />
+    </xacro:ur_robot>
+    <xacro:ur_ros2_control
+        name="$(arg ur_type)"
+        tf_prefix="$(arg ur_type)_"
+        kinematics_parameters_file="$(arg kinematics_parameters_file)"
+        robot_ip="$(arg robot_ip)"
+        script_filename="$(arg ur_script_filename)"
+        output_recipe_filename="$(arg ur_output_recipe_filename)"
+        input_recipe_filename="$(arg ur_input_recipe_filename)"
+        use_mock_hardware="$(arg use_mock_hardware)"
+        mock_sensor_commands="$(arg mock_sensor_commands)"
+        headless_mode="$(arg headless_mode)"
+    />
+</robot>
+<!-- Include your custom gripper and add the joint to connect to it, then go to the
     ur_controllers.yaml and change the ee link in the controller parameters -->
-    <!-- <xacro:include filename="$(find gripper_description)/urdf/ur_gripper.xacro" /> -->
-    <!-- <joint name="example_gripper_joint" type="fixed">
+<!-- <xacro:include filename="$(find gripper_description)/urdf/ur_gripper.xacro" /> -->
+<!-- <joint name="example_gripper_joint" type="fixed">
         <parent link="tool0" />
         <child link="gripper_link" />
         <origin xyz="0 0 0" rpy="0 0 0" />
     </joint> -->
-</robot>
